File: kicad/antenna.kicad_sch (KiCad schematic)
At the start: 40 parts, among them J1 Bus_PCI_Express_x1, J4 Conn_01x02, J6 USB_C_Receptacle_USB2.0_16P, U2 RP2040, U4 W25Q128JVP, U9 MCP25625T-E/ML, X1 ABM8-272-T3, Y2 X322516MLB4SI

Commit message: update DXF to new hole positions
Parts:
- removed D1, D2: LED, LED_SMD:LED_0603_1608Metric, symbol Device:LED
- removed R1, R2: 150, Resistor_SMD:R_0603_1608Metric, symbol Device:R
- added J5: Conn_02x08_Odd_Even, Connector_PinSocket_2.54mm:PinSocket_2x08_P2.54mm_Vertical, symbol Connector_Generic:Conn_02x08_Odd_Even
Connections:
- net CANSTBY: now also U2.38 (GPIO26_ADC0)
- net GND: now also J5.1 (Pin_1), J5.16 (Pin_16), J5.2 (Pin_2)
- new net CTS: J5.3 (Pin_3)
- new net P1.0: J5.13 (Pin_13)
- new net P1.1: J5.15 (Pin_15)
- new net P1.2: J5.14 (Pin_14)
- new net P1.3: J5.12 (Pin_12)
- new net P3.3: J5.10 (Pin_10)
- new net P3.4: J5.8 (Pin_8)
- new net RTS: J5.11 (Pin_11)
- new net RX: J5.7 (Pin_7)
- new net TX: J5.9 (Pin_9)
- new net Vcc: J5.4 (Pin_4)
- new net Vusb: J5.5 (Pin_5), J5.6 (Pin_6)
- no-connect marks 44 -> 43

Commit message: test
Other:
- note added: "test"
Changed lines of the file:
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@@
+		)
+	)
+	(text "test"
+		(exclude_from_sim no)
+		(at 150.368 310.896 0)
+		(effects
+			(font
+				(size 5.08 5.08)
+			)
 		)
 	)
@@
 	(label "USB_D2+"
 		(at 262.89 151.13 0)
-		(fields_autoplaced yes)
 		(effects
 			(font
@@
 	(label "XOUT_pre"
 		(at 179.07 273.05 180)
-		(fields_autoplaced yes)
 		(effects
 			(font
@@
 	(label "~{USB_BOOT_S}"
 		(at 74.93 167.64 0)
-		(fields_autoplaced yes)
 		(effects
 			(font
@@
 	(label "QSPI_SD3"
 		(at 260.35 173.99 0)
-		(fields_autoplaced yes)
 		(effects
 			(font
@@
 	(label "QSPI_SD1"
 		(at 109.22 175.26 0)
-		(fields_autoplaced yes)
 		(effects
 			(font
@@
 	(label "XIN"
 		(at 260.35 189.23 0)
-		(fields_autoplaced yes)
 		(effects
 			(font
@@
 	(label "USB_D+"
 		(at 241.3 147.32 0)
-		(fields_autoplaced yes)
 		(effects
 			(font
@@
 	(label "SWD"
 		(at 255.27 212.09 0)
-		(fields_autoplaced yes)
 		(effects
 			(font
@@
 	(label "QSPI_SS"
 		(at 109.22 167.64 0)
-		(fields_autoplaced yes)
 		(effects
 			(font
@@
 	(label "QSPI_SD3"
 		(at 109.22 180.34 0)
-		(fields_autoplaced yes)
 		(effects
 			(font
@@
 	(label "XIN"
 		(at 203.2 250.19 180)
-		(fields_autoplaced yes)
 		(effects
 			(font
@@
 	(label "QSPI_SD2"
 		(at 109.22 177.8 0)
-		(fields_autoplaced yes)
 		(effects
 			(font
@@
 	(label "QSPI_SS"
 		(at 260.35 161.29 0)
-		(fields_autoplaced yes)
 		(effects
 			(font
@@
 	(label "XOUT"
 		(at 204.47 273.05 180)
-		(fields_autoplaced yes)
 		(effects
 			(font
@@
 	(label "SWCLK"
 		(at 255.27 209.55 0)
-		(fields_autoplaced yes)
 		(effects
 			(font
@@
 	(label "QSPI_SCLK"
 		(at 109.22 170.18 0)
-		(fields_autoplaced yes)
 		(effects
 			(font
@@
 	(label "QSPI_SD1"
 		(at 260.35 168.91 0)
-		(fields_autoplaced yes)
 		(effects
 			(font
@@
 	(label "QSPI_SCLK"
 		(at 260.35 176.53 0)
-		(fields_autoplaced yes)
 		(effects
 			(font
@@
 	(label "USB_D-"
 		(at 241.3 156.21 0)
-		(fields_autoplaced yes)
 		(effects
 			(font
@@
 	(label "USB_D2-"
 		(at 262.89 153.67 0)
-		(fields_autoplaced yes)
 		(effects
 			(font
@@
 	(label "QSPI_SD2"
 		(at 260.35 171.45 0)
-		(fields_autoplaced yes)
 		(effects
 			(font
@@
 	(label "QSPI_SD0"
 		(at 109.22 172.72 0)
-		(fields_autoplaced yes)
 		(effects
 			(font
@@
 	(label "XOUT"
 		(at 260.35 199.39 0)
-		(fields_autoplaced yes)
 		(effects
 			(font
@@
 	(label "RUN"
 		(at 259.08 135.89 0)
-		(fields_autoplaced yes)
 		(effects
 			(font
@@
 	(label "QSPI_SD0"
 		(at 260.35 166.37 0)
-		(fields_autoplaced yes)
-		(effects
-			(font
+		(effects
+			(font
